File: bulb_driver/bulb_driver.kicad_pcb (KiCad board)
At the start: 2 copper layers, 1 part, among them U1 LM3410DGN

Commit message: Project update
Parts:
- added C1: 10u, Capacitor_SMD:C_1210_3225Metric, F.Cu at (102.0, 83.5)
- added C2: 10u, Capacitor_SMD:C_1210_3225Metric, F.Cu at (114.8, 86.5)
- added C3: 10u, Capacitor_SMD:C_1210_3225Metric, F.Cu at (105.2, 83.5)
- added C4: 10u, Capacitor_SMD:C_1210_3225Metric, F.Cu at (118.0, 86.5)
- added D1: SS34, Diode_SMD:D_SMC, F.Cu at (118.1, 80.8)
- added D2: 23V, Diode_SMD:D_SOD-123, F.Cu at (115.2, 90.0)
- added H1: M3, MountingHole:MountingHole_3.2mm_M3_Pad_Via, F.Cu at (128.5, 95.0)
- added H2: M3, MountingHole:MountingHole_3.2mm_M3_Pad_Via, F.Cu at (128.5, 70.0)
- added H3: M3, MountingHole:MountingHole_3.2mm_M3_Pad_Via, F.Cu at (90.5, 95.0)
- added H4: M3, MountingHole:MountingHole_3.2mm_M3_Pad_Via, F.Cu at (90.5, 70.0)
- added J1: PWR_IN, Connector_Wire:SolderWire-1sqmm_1x02_P7.8mm_D1.4mm_OD3.9mm, F.Cu at (90.5, 87.7)
- added J2: DIMM, Connector_PinHeader_2.54mm:PinHeader_1x02_P2.54mm_Vertical, F.Cu at (96.6, 86.7)
- added J3: LED_OUT, Connector_Wire:SolderWire-1sqmm_1x02_P7.8mm_D1.4mm_OD3.9mm, F.Cu at (128.5, 80.8)
- added L1: 150u, Inductor_SMD:L_Bourns_SRR1210A, F.Cu at (106.9, 74.5)
- added R1: 1R, Resistor_SMD:R_0805_2012Metric, F.Cu at (111.1, 88.7)
- added R2: 39R, Resistor_SMD:R_0805_2012Metric, F.Cu at (112.0, 86.0)
- added R3: 10k, Resistor_SMD:R_0805_2012Metric, F.Cu at (99.4, 83.0)
- added R4: 1R, Resistor_SMD:R_0805_2012Metric, F.Cu at (111.1, 90.6)
- U1: footprint Package_SO:TI_SO-PowerPAD-8_ThermalVias -> projectfb:HVSSOP-8-1EP_3x3mm_P0.65mm_EP1.57x1.89mm
- moved U1 62.0 mm to (110.0, 82.5)
Connections:
- U1 pad 1: (no net) -> unconnected-(U1-NC-Pad1)
- U1 pad 2: unconnected-(U1-PGND-Pad2) -> GND
- U1 pad 3: unconnected-(U1-VIN-Pad3) -> VCC
- U1 pad 4: unconnected-(U1-DIM-Pad4) -> PWM
- U1 pad 5: unconnected-(U1-FB-Pad5) -> /FEEDBACK
- U1 pad 6: unconnected-(U1-AGND-Pad6) -> GND
- U1 pad 7: unconnected-(U1-SW-Pad7) -> Net-(D1-A)
- U1 pad 8: (no net) -> unconnected-(U1-NC-Pad8)
- U1 pad 9: unconnected-(U1-DAP-Pad9) -> GND
Routing:
- net /LED+: track 0.00 -> 22.2 mm
- net /LED-: track 0.00 -> 18.4 mm
- net PWM: track 0.00 -> 11.5 mm
- net /FEEDBACK: track 0.00 -> 7.25 mm
- net GND: vias 0 -> 28
- added copper zone on F.Cu, net /LED+
- added copper zone on F.Cu, net /LED-
- added copper zone on B.Cu, net GND
- added copper zone on F.Cu, net GND
- added copper zone on F.Cu, net Net-(D1-A)
- added copper zone on F.Cu, net VCC
Other:
- board outline added: 46 x 33 mm
- board text added: "LM3410 LED Driver module Rev 1.0.0"
