File: bulb_driver/lm3410driver.kicad_sch (KiCad schematic)
At the start: 13 parts, among them J3 LED_OUT, U1 LM3410DGN

Commit message: Update LED driver schematic
Parts:
- removed C4: 10u, Capacitor_SMD:C_1210_3225Metric, symbol Device:C
- L1: value 150u -> 22u
- renumbered C3 to C1, C1 to C2, C2 to C3, R3 to R1, R1 to R3, U1 to U2
Other:
- note added: "22uH for 200mA at 22V - 4V in 8u2 for 1A at 11V - 4V in Equation (V_{in} × (V_{out} − V_{in}))/(I_{ripple%} × I_{out} × (V_{out}/V_{in}) × 525 000 × V_{out}) I_{ripple%} = 0,2 - 0,4"
- note added: "I_{out} = 0,19/R"
