File: bulb_driver/usb.kicad_sch (KiCad schematic)
At the start: 0 parts

Commit message: Update schematics
Parts:
- added J1: USB_C_Receptacle_PowerOnly_6P, symbol Connector:USB_C_Receptacle_PowerOnly_6P
Connections:
- new net: J1.A12 (GND), J1.B12 (GND)
- new net: J1.A9 (VBUS), J1.B9 (VBUS)
Other:
- note added: "add IP2312 charger schematic"
Changed lines of the file:
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@@
 	(generator_version "8.0")
 	(paper "A4")
+	(text "add  IP2312 charger schematic\n"
+		(exclude_from_sim no)
+		(at 97.282 57.404 0)
+		(effects
+			(font
+				(size 1.27 1.27)
+			)
+		)
+	)
+	(symbol
+		(lib_id "Connector:USB_C_Receptacle_PowerOnly_6P")
+		(at 63.5 63.5 0)
+		(unit 1)
+		(exclude_from_sim no)
+		(in_bom yes)
+		(on_board yes)
+		(dnp no)
+		(fields_autoplaced yes)
+		(property "Reference" "J1"
+			(at 63.5 45.72 0)
+			(effects
+				(font
+					(size 1.27 1.27)
+				)
+			)
+		)
+		(property "Value" "USB_C_Receptacle_PowerOnly_6P"
+			(at 63.5 48.26 0)
+			(effects
+				(font
+					(size 1.27 1.27)
+				)
+			)
+		)
+		(property "Footprint" ""
+			(at 67.31 60.96 0)
+			(effects
+				(font
+					(size 1.27 1.27)
+				)
+				(hide yes)
+			)
+		)
+		(property "Datasheet" "https://www.usb.org/sites/default/files/documents/usb_type-c.zip"
+			(at 63.5 63.5 0)
+			(effects
+				(font
+					(size 1.27 1.27)
+				)
+				(hide yes)
+			)
+		)
+		(property "Description" "USB Power-Only 6P Type-C Receptacle connector"
+			(at 63.5 63.5 0)
+			(effects
+				(font
+					(size 1.27 1.27)
+				)
+				(hide yes)
+			)
+		)
+		(pin "A12"
+		)
+		(pin "B9"
+		)
+		(pin "A5"
+		)
+		(pin "A9"
+		)
+		(pin "S1"
+		)
+		(pin "B12"
+		)
+		(pin "B5"
+		)
+		(instances
+			(project ""
+				(path "/a662f7bf-9c13-4ccb-87cd-8868bb64c17e/50adb9b4-1b65-4ec0-8512-a06bfbe73499"
+					(reference "J1")
+					(unit 1)
+				)
+			)
+		)
+	)
 )
